File: SimonSays/_autosave-SimonSays.kicad_sch (KiCad schematic)
At the start: 22 parts, among them X1 Crystal

Commit message: Added
Parts:
- D1: value Blue -> Yellow
- D2: value Yellow -> Blue
- D3: value Red -> Green
- D4: value Green -> Red
Connections:
- net GNDREF: now also 5V1.2 (-)
- net at D1.2 (A): now also UIntegratedCircuit1.11 (PD5); no longer UIntegratedCircuit1.12 (PD6)
- net at 5V1.1 (+), R9.2, UIntegratedCircuit1.7 (VCC): now also UIntegratedCircuit1.20 (AVCC)
- net at S1.8: now also UIntegratedCircuit1.12 (PD6)
Changed lines of the file:
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@@
   (junction (at 166.116 116.459) (diameter 0) (color 0 0 0 0)
   )
-  (junction (at 157.226 57.658) (diameter 0) (color 0 0 0 0)
-  )
   (junction (at 74.422 90.17) (diameter 0) (color 0 0 0 0)
   )
+  (junction (at 112.776 110.109) (diameter 0) (color 0 0 0 0)
+  )
   (junction (at 112.776 134.874) (diameter 0) (color 0 0 0 0)
   )
@@
   (junction (at 161.036 124.079) (diameter 0) (color 0 0 0 0)
   )
-  (junction (at 112.776 110.109) (diameter 0) (color 0 0 0 0)
-  )
   (junction (at 154.432 133.35) (diameter 0) (color 0 0 0 0)
   )
@@
     (stroke (width 0) (type default) (color 0 0 0 0))
   )
-  (wire (pts (xy 115.316 111.76) (xy 103.632 111.76))
+  (wire (pts (xy 103.632 111.76) (xy 117.856 111.76))
     (stroke (width 0) (type default) (color 0 0 0 0))
   )
@@
     (stroke (width 0) (type default) (color 0 0 0 0))
   )
+  (wire (pts (xy 112.776 109.22) (xy 112.776 110.109))
+    (stroke (width 0) (type default) (color 0 0 0 0))
+  )
   (wire (pts (xy 168.656 108.712) (xy 185.42 108.712))
     (stroke (width 0) (type default) (color 0 0 0 0))
@@
     (stroke (width 0) (type default) (color 0 0 0 0))
   )
-  (wire (pts (xy 115.316 86.614) (xy 115.316 111.76))
+  (wire (pts (xy 115.316 86.614) (xy 115.316 109.22))
     (stroke (width 0) (type default) (color 0 0 0 0))
   )
@@
     (stroke (width 0) (type default) (color 0 0 0 0))
   )
-  (wire (pts (xy 157.226 40.894) (xy 157.226 57.658))
+  (wire (pts (xy 157.226 40.894) (xy 157.226 54.864))
     (stroke (width 0) (type default) (color 0 0 0 0))
   )
@@
     (stroke (width 0) (type default) (color 0 0 0 0))
   )
+  (wire (pts (xy 117.856 86.614) (xy 117.856 111.76))
+    (stroke (width 0) (type default) (color 0 0 0 0))
+  )
   (wire (pts (xy 117.856 117.729) (xy 117.856 125.222))
     (stroke (width 0) (type default) (color 0 0 0 0))
@@
     (stroke (width 0) (type default) (color 0 0 0 0))
   )
-  (wire (pts (xy 157.226 57.658) (xy 184.15 57.658))
-    (stroke (width 0) (type default) (color 0 0 0 0))
-  )
   (wire (pts (xy 190.5 116.078) (xy 190.5 116.205))
     (stroke (width 0) (type default) (color 0 0 0 0))
@@
     (stroke (width 0) (type default) (color 0 0 0 0))
   )
-  (wire (pts (xy 153.416 54.864) (xy 187.198 54.864))
-    (stroke (width 0) (type default) (color 0 0 0 0))
-  )
   (wire (pts (xy 137.16 133.858) (xy 137.16 133.985))
     (stroke (width 0) (type default) (color 0 0 0 0))
@@
     (stroke (width 0) (type default) (color 0 0 0 0))
   )
-  (wire (pts (xy 112.776 86.868) (xy 112.776 110.109))
-    (stroke (width 0) (type default) (color 0 0 0 0))
-  )
   (wire (pts (xy 153.416 40.894) (xy 145.034 40.894))
     (stroke (width 0) (type default) (color 0 0 0 0))
@@
     (stroke (width 0) (type default) (color 0 0 0 0))
   )
+  (wire (pts (xy 115.316 109.22) (xy 112.776 109.22))
+    (stroke (width 0) (type default) (color 0 0 0 0))
+  )
   (wire (pts (xy 112.776 134.62) (xy 112.776 134.874))
     (stroke (width 0) (type default) (color 0 0 0 0))
@@
     (stroke (width 0) (type default) (color 0 0 0 0))
   )
-  (wire (pts (xy 112.776 110.109) (xy 112.776 110.744))
+  (wire (pts (xy 112.776 110.109) (xy 112.776 111.506))
     (stroke (width 0) (type default) (color 0 0 0 0))
   )
@@
     (stroke (width 0) (type default) (color 0 0 0 0))
   )
-  (wire (pts (xy 145.034 57.658) (xy 157.226 57.658))
+  (wire (pts (xy 145.034 57.658) (xy 184.15 57.658))
     (stroke (width 0) (type default) (color 0 0 0 0))
   )
@@
   )
   (wire (pts (xy 161.036 123.698) (xy 161.036 124.079))
+    (stroke (width 0) (type default) (color 0 0 0 0))
+  )
+  (wire (pts (xy 187.198 54.864) (xy 157.226 54.864))
     (stroke (width 0) (type default) (color 0 0 0 0))
   )
@@
       (effects (font (size 1.27 1.27)) (justify right))
     )
-    (property "Value" "Blue" (id 1) (at 96.012 119.888 90)
+    (property "Value" "Yellow" (id 1) (at 96.012 119.888 90)
       (effects (font (size 1.27 1.27)) (justify right))
     )
@@
       (effects (font (size 1.27 1.27)) (justify right))
     )
-    (property "Value" "Green" (id 1) (at 171.45 118.872 90)
+    (property "Value" "Red" (id 1) (at 171.45 118.872 90)
       (effects (font (size 1.27 1.27)) (justify right))
     )
@@
       (effects (font (size 1.27 1.27)) (justify right))
     )
-    (property "Value" "Yellow" (id 1) (at 122.936 119.888 90)
+    (property "Value" "Blue" (id 1) (at 122.936 119.888 90)
       (effects (font (size 1.27 1.27)) (justify right))
     )
@@
     (pin "2")
   )
+  (symbol (lib_id "power:GNDREF") (at 153.416 54.864 0) (unit 1)
+    (in_bom yes) (on_board yes) (fields_autoplaced)
+    (property "Reference" "#PWR?" (id 0) (at 153.416 61.214 0)
+      (effects (font (size 1.27 1.27)) hide)
+    )
+    (property "Value" "GNDREF" (id 1) (at 153.416 59.69 0))
+    (property "Footprint" "" (id 2) (at 153.416 54.864 0)
+      (effects (font (size 1.27 1.27)) hide)
+    )
+    (property "Datasheet" "" (id 3) (at 153.416 54.864 0)
+      (effects (font (size 1.27 1.27)) hide)
+    )
+    (pin "1")
+  )
   (symbol (lib_id "Device:LED") (at 154.432 116.332 90) (unit 1)
     (in_bom yes) (on_board yes)
@@
       (effects (font (size 1.27 1.27)) (justify right))
     )
-    (property "Value" "Red" (id 1) (at 148.844 119.126 90)
+    (property "Value" "Green" (id 1) (at 148.844 119.126 90)
       (effects (font (size 1.27 1.27)) (justify right))
     )
@@
       (reference "#PWR0109") (unit 1) (value "GNDREF") (footprint "")
     )
+    (path "/a1434e3b-aba4-410a-858d-823582b176a7"
+      (reference "#PWR?") (unit 1) (value "GNDREF") (footprint "")
+    )
     (path "/672cce20-82ef-4cef-a268-b67f5ebf55d6"
       (reference "5V1") (unit 1) (value "Battery_Cell") (footprint "Battery:BatteryHolder_Bulgin_BX0036_1xC")
@@
     )
     (path "/0be4244f-8e96-4893-a299-e98dc8d4f872"
-      (reference "D1") (unit 1) (value "Blue") (footprint "")
+      (reference "D1") (unit 1) (value "Yellow") (footprint "")
     )
     (path "/91729398-e312-40e3-923a-85ad380afa7a"
-      (reference "D2") (unit 1) (value "Yellow") (footprint "")
+      (reference "D2") (unit 1) (value "Blue") (footprint "")
     )
     (path "/a93f1b2c-885b-45fb-95cb-cee2cf6e14d2"
-      (reference "D3") (unit 1) (value "Red") (footprint "")
+      (reference "D3") (unit 1) (value "Green") (footprint "")
     )
     (path "/3ec61d98-ee61-475a-a9c1-9662d4842c34"
-      (reference "D4") (unit 1) (value "Green") (footprint "")
+      (reference "D4") (unit 1) (value "Red") (footprint "")
     )
     (path "/e962bc73-4e3b-4fbe-90ec-ef049ff02d8b"
